File: WeeKeys.kicad_sch (KiCad schematic)
At the start: 0 parts

Commit message: Add files via upload
Parts:
- added D1: L08R5000Q1, L08R5000Q1:LEDRD254W57D500H1070, symbol L08R5000Q1:L08R5000Q1
- added R1: R, symbol Device:R
- added SW1, SW2, SW3, SW4: SW_Push, symbol Switch:SW_Push
- added U1: XIAO-RP2040-DIP, Module:MOUDLE14P-XIAO-DIP-SMD, symbol Seeed_Studio_XIAO_Series:XIAO-RP2040-DIP
Connections:
- new net: D1.A, R1.1
- new net Button1: SW1.1, U1.1 (GPIO26/ADC0/A0)
- new net Button2: SW3.1, U1.2 (GPIO27/ADC1/A1)
- new net Button3: SW2.1, U1.3 (GPIO28/ADC2/A2)
- new net Button4: SW4.1, U1.4 (GPIO29/ADC3/A3)
- new net GND: D1.C, SW1.2, SW2.2, SW3.2, SW4.2, U1.13 (GND)
- new net Led: R1.2, U1.5 (GPIO6/SDA)

Commit message: Add files via upload
Parts:
- D1: footprint L08R5000Q1:LEDRD254W57D500H1070 -> Footprints:LEDRD254W57D500H1070
- R1: footprint (none) -> Resistor_THT:R_Axial_DIN0204_L3.6mm_D1.6mm_P5.08mm_Horizontal
- SW1, SW2, SW3, SW4: footprint (none) -> Button_Switch_Keyboard:SW_Cherry_MX_1.00u_PCB
- U1: footprint Module:MOUDLE14P-XIAO-DIP-SMD -> Footprints:XIAO-RP2040-DIP (2)
Changed lines of the file:
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@@
 			)
 		)
-		(property "Footprint" ""
+		(property "Footprint" "Button_Switch_Keyboard:SW_Cherry_MX_1.00u_PCB"
 			(at 181.61 78.74 0)
 			(effects
@@
 			)
 		)
-		(property "Footprint" "L08R5000Q1:LEDRD254W57D500H1070"
+		(property "Footprint" "Footprints:LEDRD254W57D500H1070"
 			(at 143.51 48.26 0)
 			(effects
@@
 			)
 		)
-		(property "Footprint" ""
+		(property "Footprint" "Button_Switch_Keyboard:SW_Cherry_MX_1.00u_PCB"
 			(at 181.61 68.58 0)
 			(effects
@@
 			)
 		)
-		(property "Footprint" ""
+		(property "Footprint" "Button_Switch_Keyboard:SW_Cherry_MX_1.00u_PCB"
 			(at 199.39 68.58 0)
 			(effects
@@
 			)
 		)
-		(property "Footprint" "Module:MOUDLE14P-XIAO-DIP-SMD"
+		(property "Footprint" "Footprints:XIAO-RP2040-DIP (2)"
 			(at 142.748 94.488 0)
 			(effects
@@
 			)
 		)
-		(property "Footprint" ""
+		(property "Footprint" "Button_Switch_Keyboard:SW_Cherry_MX_1.00u_PCB"
 			(at 200.66 78.74 0)
 			(effects
@@
 			)
 		)
-		(property "Footprint" ""
+		(property "Footprint" "Resistor_THT:R_Axial_DIN0204_L3.6mm_D1.6mm_P5.08mm_Horizontal"
 			(at 134.112 52.07 90)
 			(effects
